Commit message: data pipeline

File: arm3dof/urdf/arm3dof.urdf (robot description, URDF)
Before this commit: robot arm3dof, 4 links, 3 joints
Joints:
- joint link1_link2: origin xyz=0 0.05 0 rpy=1.5707963267949 1.5707963267949 0 -> xyz=0 0.05 0 rpy=1.5707963267949 1.5707963267949 -1.5707963267949

Commit message: urdfpy+open3d pipeline

File: arm3dof/urdf/arm3dof.urdf (robot description, URDF)
Before this commit: robot arm3dof, 4 links, 3 joints
Links:
- link base: geometry collision mesh filename=../meshes/base.STL; visual mesh filename=../meshes/base.STL
- link link1: geometry collision mesh filename=../meshes/link1.STL; visual mesh filename=../meshes/link1.STL
- link link2: geometry collision mesh filename=../meshes/link2.STL; visual mesh filename=../meshes/link2.STL
- link link3: geometry collision mesh filename=../meshes/link3.STL; visual mesh filename=../meshes/link3.STL
