Commit message: delete

File: arm4dof/urdf/arm4dof.urdf (robot description, URDF)
Before this commit: robot arm4dof, 5 links, 4 joints
Joints:
- joint base_l0: origin xyz=0 0 0.068 rpy=1.5707963267949 0 1.5707963267949 -> xyz=0 0 0.068 rpy=1.5707963267949 0 0
- joint l1_l2: origin xyz=0 0.04 -0.00129999999999999 rpy=1.5707963267949 1.5707963267949 0 -> xyz=0 0.04 -0.00129999999999999 rpy=-1.5707963267949 -1.5707963267949 0
