Commit message: add a sphere fixed link for cetner calculation

File: 4dof_2nd/urdf/4dof_2nd.urdf (robot description, URDF)
Before this commit: robot 4dof_2nd, 5 links, 4 joints
Links:
- added link sphere_link, mass 0.005; collision sphere radius=0.02; visual sphere radius=0.02
Joints:
- added joint L4_sphere_joint: type fixed, parent L4, child sphere_link, origin xyz=0 0 0.06 rpy=0 0 0
